Commit message: visualization and collision meshes for abb_6700_175_305

File: abb_irb6700_support/urdf/irb6700_175_305_macro.xacro (robot description, xacro)
@@ -163,5 +163,5 @@
     </joint>
     <joint name="${prefix}joint_3" type="revolute">
-      <origin xyz="0 0 1.125" rpy="0 0 0" />
+      <origin xyz="0 0 1.135" rpy="0 0 0" />
       <parent link="${prefix}link_2" />
       <child link="${prefix}link_3" />
@@ -177,5 +177,5 @@
     </joint>
     <joint name="${prefix}joint_5" type="revolute">
-      <origin xyz="1.1425 0 0" rpy="0 0 0" />
+      <origin xyz="1.593 0 0" rpy="0 0 0" />
       <parent link="${prefix}link_4" />
       <child link="${prefix}link_5" />
